File: BUS_ORIC/Extensions/RTC/Kicad5/RTC.kicad_pcb (KiCad board)
At the start: 2 copper layers, 76.2 x 49.5 mm, 15 parts, among them J1 SLOT1, U1 ICM7170, U2 GAL16V8, Y1 32.768kHz

Commit message: Add files via upload
Routing:
- net /D4: track 38.4 -> 39.3 mm
